Commit message: Aapted physics parameters

File: simple_test/deformable_object/CubePrismatic/cube_prismatic_left.urdf (robot description, URDF)
Before this commit: robot urdf_robot, 5 links, 4 joints
Links:
- link panda_hand: mass .81 -> 0.81
- link panda_leftfinger: mass 0.1 -> 0.81
- link panda_rightfinger: mass 0.1 -> 0.81
Joints:
- joint panda_finger_joint1: limit lower=0.0 upper=0.04 effort=20 velocity=0.2 -> lower=0.0 upper=0.04 effort=200 velocity=0.2
- joint panda_finger_joint2: limit lower=0.0 upper=0.04 effort=20 velocity=0.2 -> lower=0.0 upper=0.04 effort=200 velocity=0.2; mimic joint=panda_finger_joint1 -> (none)

Commit message: Modified physics parameters

File: simple_test/deformable_object/CubePrismatic/cube_prismatic_left.urdf (robot description, URDF)
Before this commit: robot urdf_robot, 5 links, 4 joints
Links:
- link panda_hand: mass 0.81 -> 20.81; geometry collision box size=0.07 .1 .1; visual box size=0.07 .1 .1
- link panda_leftfinger: mass 0.81 -> 10; geometry collision box size=0.07 .02 .1; visual box size=0.07 .02 .1
- link panda_rightfinger: mass 0.81 -> 10; geometry collision box size=0.07 .02 .1; visual box size=0.07 .02 .1
