Commit message: Added version with new gripper position

File: simple_test/deformable_object/CubePrismatic/cube_prismatic_right.urdf (robot description, URDF)
Before this commit: robot urdf_robot, 5 links, 4 joints
Joints:
- joint panda_hand_joint: origin xyz=-0.8 0 -0.06 rpy=0 -1.57 0.0 -> xyz=-0.9 0 0.03 rpy=3.14 0.0 0.0
